Commit message: feat(twin): update URDF and virtual ToF/IR sensors
Keeps the digital twin in sync with the real arm: refreshed URDF
link geometry and virtual sensor models updated to match the
VL53L5CX grid and NOR-inverted IR behavior.

File: braccio_main_runner/braccio_twin/urdf/braccio.urdf (robot description, URDF)
Before this commit: robot braccio_v2, 15 links, 14 joints
Links:
- removed link tof_back_link
- removed link tof_front_link
- added link tof_left_link, mass 0.001
- added link tof_right_link, mass 0.001
Joints:
- removed joint mount_tof_back
- removed joint mount_tof_front
- added joint mount_tof_left: type fixed, parent wrist_roll_link, child tof_left_link, origin xyz=0.010 0.025 0 rpy=0 0 1.5708
- added joint mount_tof_right: type fixed, parent wrist_roll_link, child tof_right_link, origin xyz=0.010 -0.025 0 rpy=0 0 -1.5708
